File: 5x5_LED_matrix.kicad_pcb (KiCad board)
At the start: 2 copper layers, 40 x 40 mm, 31 parts

Commit message: Major change close to final.
Parts:
- removed A+, B+, C+: +, connector_ext:SMD_1P_2.8x2.0
- removed A-, B-, C-: -, connector_ext:SMD_1P_2.8x2.0
- added 1+: +, connector_ext:SMD_1P_2.8x2.0, F.Cu at (125.7, 101.5)
- added 1-: -, connector_ext:SMD_1P_2.8x2.0, F.Cu at (125.7, 114.5)
- added 2+: +, connector_ext:SMD_1P_2.8x2.0, F.Cu at (118.6, 94.4)
- added 2-: -, connector_ext:SMD_1P_2.8x2.0, F.Cu at (118.6, 121.5)
- added 3+: +, connector_ext:SMD_1P_2.8x2.0, F.Cu at (112.1, 94.4)
- added 3-: -, connector_ext:SMD_1P_2.8x2.0, F.Cu at (112.1, 121.5)
- added 4+: +, connector_ext:SMD_1P_2.8x2.0, F.Cu at (105.6, 94.4)
- added 4-: -, connector_ext:SMD_1P_2.8x2.0, F.Cu at (105.6, 121.5)
- added 5+: +, connector_ext:SMD_1P_2.8x2.0, F.Cu at (98.5, 101.5)
- added 5-: -, connector_ext:SMD_1P_2.8x2.0, F.Cu at (98.5, 114.5)
- D12, D14: footprint OSRAM:LED-GWCSSRM2.CM_OSRAM -> OSRAM:LED-SFH4776_OSRAM_fit
- moved D15 11.1 mm to (112.1, 115.8), turned to 270 degrees
- moved D3 11.1 mm to (119.9, 108.0), turned to 180 degrees
- moved D11 11.1 mm to (112.1, 100.2), turned to 270 degrees
- moved D23 11.0 mm to (104.3, 108.0), turned to 0 degrees
- moved D25 10.9 mm to (106.9, 113.5), turned to 270 degrees
- moved D1 10.9 mm to (117.3, 102.4), turned to 270 degrees
- moved D5 10.9 mm to (117.3, 113.5), turned to 270 degrees
- moved D21 10.8 mm to (106.9, 102.4), turned to 270 degrees
- moved D2 10.6 mm to (118.6, 105.3), turned to 0 degrees
- moved D24 10.6 mm to (105.6, 110.5), turned to 0 degrees
- moved D22 10.4 mm to (105.6, 105.3), turned to 180 degrees
- moved D4 10.4 mm to (118.6, 110.5), turned to 180 degrees
- moved D10 10.3 mm to (114.7, 114.7), turned to 270 degrees
- moved D16 10.3 mm to (109.5, 101.2), turned to 270 degrees
- moved D6 10.3 mm to (114.7, 101.2), turned to 270 degrees
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Connections:
- D21 pad 2: Net-(D16-Pad2) -> Net-(D21-Pad2)
- D25 pad 1: Net-(D20-Pad1) -> Net-(D25-Pad1)
- D5 pad 1: Net-(D10-Pad1) -> Net-(D5-Pad1)
- D6 pad 2: Net-(D1-Pad2) -> Net-(D6-Pad2)
Routing:
- added copper zone on F.Cu, net Net-(D21-Pad2)
- added copper zone on F.Cu, net Net-(D25-Pad1)
- added copper zone on F.Cu, net Net-(D5-Pad1)
- added copper zone on F.Cu, net Net-(D6-Pad2)
Other:
- outline, holes or cut-outs redrawn
- board text added: "SFH4776 x 24, GW_CSSRM2.CM x 1 20200428"
- board text removed: "3 x GW CSSRM2.CM, and 22 x SFH 4776 LED Matrix, ver. 0.5.0.(2019-05-23) Assemblied by TODDY Korea Inc. Designed by Hoyoung Lee."
