File: 5x5_LED_matrix.sch (KiCad schematic (older format))
At the start: 31 parts, among them J1 +, J2 -, J3 +, J4 -, J5 +, J6 -

Commit message: Major change close to final.
Parts:
- added J1, J9: +, connector_ext:SMD_1P_2.8x2.0, symbol Connector_Generic:Conn_01x01
- added J10, J2: -, connector_ext:SMD_1P_2.8x2.0, symbol Connector_Generic:Conn_01x01
- D12, D14: value GW_CSSRM2.CM -> SFH4776; footprint OSRAM:LED-GWCSSRM2.CM_OSRAM -> OSRAM:LED-SFH4776_OSRAM_fit
- renumbered J1 to J3, J2 to J4, J3 to J5, J4 to J6, J5 to J7, J6 to J8
Connections:
- net at D6.2 (A), J3.1 (Pin_1): no longer D1.2 (A)
- net at D16.2 (A), J7.1 (Pin_1): no longer D21.2 (A)
- net at D10.1 (K), J4.1 (Pin_1): no longer D5.1 (K)
- net at D20.1 (K), J8.1 (Pin_1): no longer D25.1 (K)
- new net: D5.1 (K), J2.1 (Pin_1)
- new net: D25.1 (K), J10.1 (Pin_1)
- new net: D1.2 (A), J1.1 (Pin_1)
- new net: D21.2 (A), J9.1 (Pin_1)
Changed lines of the file:
@@
 EESchema Schematic File Version 4
-LIBS:5x5_LED_matrix-cache
-EELAYER 29 0
+EELAYER 30 0
 EELAYER END
 $Descr A4 11693 8268
@@
 $EndComp
 $Comp
-L Connector_Generic:Conn_01x01 J1
+L Connector_Generic:Conn_01x01 J3
 U 1 1 5C965BD7
 P 2700 3200
-F 0 "J1" H 2600 3050 50  0000 C CNN
+F 0 "J3" H 2600 3050 50  0000 C CNN
 F 1 "+" H 2650 3300 50  0000 C CNN
 F 2 "connector_ext:SMD_1P_2.8x2.0" H 2700 3200 50  0001 C CNN
@@
 $EndComp
 $Comp
-L Connector_Generic:Conn_01x01 J3
+L Connector_Generic:Conn_01x01 J5
 U 1 1 5C965DD9
 P 2700 3600
-F 0 "J3" H 2600 3450 50  0000 C CNN
+F 0 "J5" H 2600 3450 50  0000 C CNN
 F 1 "+" H 2650 3700 50  0000 C CNN
 F 2 "connector_ext:SMD_1P_2.8x2.0" H 2700 3600 50  0001 C CNN
@@
 $EndComp
 $Comp
-L Connector_Generic:Conn_01x01 J5
+L Connector_Generic:Conn_01x01 J7
 U 1 1 5C966064
 P 2700 4000
-F 0 "J5" H 2600 3850 50  0000 C CNN
+F 0 "J7" H 2600 3850 50  0000 C CNN
 F 1 "+" H 2650 4100 50  0000 C CNN
 F 2 "connector_ext:SMD_1P_2.8x2.0" H 2700 4000 50  0001 C CNN
@@
 $EndComp
 $Comp
-L Connector_Generic:Conn_01x01 J2
+L Connector_Generic:Conn_01x01 J4
 U 1 1 5C9660F8
 P 6600 3200
-F 0 "J2" H 6680 3242 50  0000 L CNN
+F 0 "J4" H 6680 3242 50  0000 L CNN
 F 1 "-" H 6680 3151 50  0000 L CNN
 F 2 "connector_ext:SMD_1P_2.8x2.0" H 6600 3200 50  0001 C CNN
@@
 $EndComp
 $Comp
-L Connector_Generic:Conn_01x01 J4
+L Connector_Generic:Conn_01x01 J6
 U 1 1 5C9662AF
 P 6600 3600
-F 0 "J4" H 6680 3642 50  0000 L CNN
+F 0 "J6" H 6680 3642 50  0000 L CNN
 F 1 "-" H 6680 3551 50  0000 L CNN
 F 2 "connector_ext:SMD_1P_2.8x2.0" H 6600 3600 50  0001 C CNN
@@
 $EndComp
 $Comp
-L Connector_Generic:Conn_01x01 J6
+L Connector_Generic:Conn_01x01 J8
 U 1 1 5C966395
 P 6600 4000
-F 0 "J6" H 6680 4042 50  0000 L CNN
+F 0 "J8" H 6680 4042 50  0000 L CNN
 F 1 "-" H 6680 3951 50  0000 L CNN
 F 2 "connector_ext:SMD_1P_2.8x2.0" H 6600 4000 50  0001 C CNN
@@
 P 4000 3600
 F 0 "D12" H 4000 3450 50  0000 C CNN
-F 1 "GW_CSSRM2.CM" H 4000 3700 50  0000 C CNN
-F 2 "OSRAM:LED-GWCSSRM2.CM_OSRAM" H 4000 3600 50  0001 C CNN
+F 1 "SFH4776" H 4000 3700 50  0000 C CNN
+F 2 "OSRAM:LED-SFH4776_OSRAM_fit" H 4000 3600 50  0001 C CNN
 F 3 "~" H 4000 3600 50  0001 C CNN
 	1    4000 3600
@@
 P 5300 3600
 F 0 "D14" H 5300 3450 50  0000 C CNN
-F 1 "GW_CSSRM2.CM" H 5300 3700 50  0000 C CNN
-F 2 "OSRAM:LED-GWCSSRM2.CM_OSRAM" H 5300 3600 50  0001 C CNN
+F 1 "SFH4776" H 5300 3700 50  0000 C CNN
+F 2 "OSRAM:LED-SFH4776_OSRAM_fit" H 5300 3600 50  0001 C CNN
 F 3 "~" H 5300 3600 50  0001 C CNN
 	1    5300 3600
@@
 $EndComp
 Wire Wire Line
-	3200 2800 3050 2800
-Wire Wire Line
-	3050 2800 3050 3200
-Wire Wire Line
-	3050 3200 3200 3200
-Wire Wire Line
-	2900 3200 3050 3200
-Connection ~ 3050 3200
+	3200 2800 2900 2800
 Wire Wire Line
 	2900 3600 3200 3600
 Wire Wire Line
-	2900 4000 3050 4000
-Wire Wire Line
-	3050 4000 3050 4400
-Wire Wire Line
-	3050 4400 3200 4400
-Connection ~ 3050 4000
-Wire Wire Line
-	3050 4000 3200 4000
+	2900 4400 3200 4400
 Wire Wire Line
 	3500 2800 3850 2800
@@
 	5450 4400 5800 4400
 Wire Wire Line
-	6100 2800 6250 2800
-Wire Wire Line
-	6250 2800 6250 3200
-Wire Wire Line
-	6250 3200 6100 3200
-Connection ~ 6250 3200
-Wire Wire Line
-	6250 4000 6250 4400
-Wire Wire Line
-	6250 4400 6100 4400
-Connection ~ 6250 4000
-Wire Wire Line
-	6250 4000 6100 4000
-Wire Wire Line
-	6250 3200 6400 3200
+	6100 2800 6400 2800
+Wire Wire Line
+	6400 4400 6100 4400
 Wire Wire Line
 	6100 3600 6400 3600
 Wire Wire Line
-	6250 4000 6400 4000
+	2900 3200 3200 3200
+$Comp
+L Connector_Generic:Conn_01x01 J1
+U 1 1 5EA808FC
+P 2700 2800
+F 0 "J1" H 2600 2650 50  0000 C CNN
+F 1 "+" H 2650 2900 50  0000 C CNN
+F 2 "connector_ext:SMD_1P_2.8x2.0" H 2700 2800 50  0001 C CNN
+F 3 "~" H 2700 2800 50  0001 C CNN
+	1    2700 2800
+	-1   0    0    1
+$EndComp
+Wire Wire Line
+	2900 4000 3200 4000
+Wire Wire Line
+	6100 3200 6400 3200
+$Comp
+L Connector_Generic:Conn_01x01 J2
+U 1 1 5EA82435
+P 6600 2800
+F 0 "J2" H 6680 2842 50  0000 L CNN
+F 1 "-" H 6680 2751 50  0000 L CNN
+F 2 "connector_ext:SMD_1P_2.8x2.0" H 6600 2800 50  0001 C CNN
+F 3 "~" H 6600 2800 50  0001 C CNN
+	1    6600 2800
+	1    0    0    -1
+$EndComp
+Wire Wire Line
+	6100 4000 6400 4000
+$Comp
+L Connector_Generic:Conn_01x01 J10
+U 1 1 5EA82C0C
+P 6600 4400
+F 0 "J10" H 6680 4442 50  0000 L CNN
+F 1 "-" H 6680 4351 50  0000 L CNN
+F 2 "connector_ext:SMD_1P_2.8x2.0" H 6600 4400 50  0001 C CNN
+F 3 "~" H 6600 4400 50  0001 C CNN
+	1    6600 4400
+	1    0    0    -1
+$EndComp
+$Comp
+L Connector_Generic:Conn_01x01 J9
+U 1 1 5EA8313A
+P 2700 4400
+F 0 "J9" H 2600 4250 50  0000 C CNN
+F 1 "+" H 2650 4500 50  0000 C CNN
+F 2 "connector_ext:SMD_1P_2.8x2.0" H 2700 4400 50  0001 C CNN
+F 3 "~" H 2700 4400 50  0001 C CNN
+	1    2700 4400
+	-1   0    0    1
+$EndComp
 $EndSCHEMATC
